File: eagle-files/SmartOutlet/ButtonLedBoard.brd (EAGLE design)
At the start: 20 x 9 mm, 6 parts, among them J1 826629-4

Commit message: Updated PCB design
Connections:
- net BLUE: now also J1.3; no longer J1.2
- net BUTTON: now also J1.2; no longer J1.4
- net GREEN: now also J1.4; no longer J1.3
Routing:
- net BLUE: track 11.3 -> 7.54 mm, vias 2 -> 0
- net BUTTON: track 3.83 -> 7.42 mm
- net GREEN: track 10.1 -> 12.2 mm
Other:
- board text added: "BLUE"
- board text added: "BUTTON"
- board text added: "GND"
- board text added: "GREEN"
Changed lines of the file:
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@@
 <drawing>
 <settings>
-<setting alwaysvectorfont="no"/>
+<setting alwaysvectorfont="yes"/>
 <setting verticaltext="up"/>
 </settings>
@@
 <wire x1="16.008" y1="8.993" x2="16.008" y2="7.493" width="0.001" layer="20"/>
 <text x="8.89" y="1.27" size="0.635" layer="21">Button</text>
+<text x="16.383" y="6.096" size="0.6096" layer="21">BLUE</text>
+<text x="3.937" y="6.096" size="0.6096" layer="21" align="bottom-right">GREEN</text>
+<text x="5.969" y="5.969" size="0.6096" layer="22" rot="MR90" align="bottom-right">GND</text>
+<text x="8.509" y="5.969" size="0.6096" layer="22" rot="MR90" align="bottom-right">BUTTON</text>
+<text x="11.049" y="5.969" size="0.6096" layer="22" rot="MR90" align="bottom-right">BLUE</text>
+<text x="13.589" y="6.096" size="0.6096" layer="22" rot="MR90" align="bottom-right">GREEN</text>
 </plain>
 <attributes>
@@
 <attribute name="POPULARITY" value="70" x="3.302" y="4.445" size="1.778" layer="27" rot="R270" display="off"/>
 <attribute name="SPICEPREFIX" value="R" x="3.302" y="4.445" size="1.778" layer="27" rot="R270" display="off"/>
-<attribute name="VALUE" x="3.556" y="2.667" size="0.635" layer="21" rot="R180"/>
+<attribute name="VALUE" x="2.286" y="2.794" size="0.635" layer="21" rot="R180"/>
 </element>
 <element name="R15" library="rcl" library_urn="urn:adsk.eagle:library:334" package="R0603" package3d_urn="urn:adsk.eagle:package:23555/3" value="1k" x="16.637" y="4.445" smashed="yes" rot="R270">
 <attribute name="POPULARITY" value="70" x="16.637" y="4.445" size="1.778" layer="27" rot="R270" display="off"/>
 <attribute name="SPICEPREFIX" value="R" x="16.637" y="4.445" size="1.778" layer="27" rot="R270" display="off"/>
-<attribute name="VALUE" x="17.018" y="2.667" size="0.635" layer="27" rot="R180"/>
+<attribute name="VALUE" x="18.542" y="2.794" size="0.635" layer="21" rot="R180"/>
 </element>
 <element name="S1" library="SparkFun-Switches" library_urn="urn:adsk.eagle:library:23465006" package="TACTILE_SWITCH_SMD_6.0X3.5MM" package3d_urn="urn:adsk.eagle:package:36446722/3" value="MOMENTARY-SWITCH-SPST-SMD-6.0X3.5MM" x="10.033" y="3.937" smashed="yes">
@@
 <signal name="BUTTON">
 <contactref element="S1" pad="2"/>
-<contactref element="J1" pad="4"/>
 <wire x1="13.183" y1="3.937" x2="13.843" y2="4.597" width="0.254" layer="1"/>
-<wire x1="13.843" y1="4.597" x2="13.843" y2="7.493" width="0.254" layer="1"/>
+<contactref element="J1" pad="2"/>
+<wire x1="13.183" y1="3.937" x2="11.303" y2="3.937" width="0.254" layer="1"/>
+<wire x1="8.763" y1="6.477" x2="8.763" y2="7.493" width="0.254" layer="1"/>
+<wire x1="11.303" y1="3.937" x2="8.763" y2="6.477" width="0.254" layer="1"/>
 </signal>
 <signal name="GND">
@@
 <signal name="GREEN">
 <contactref element="R14" pad="2"/>
-<contactref element="J1" pad="3"/>
 <wire x1="3.302" y1="3.595" x2="3.722" y2="3.595" width="0.254" layer="1"/>
 <wire x1="3.722" y1="3.595" x2="4.572" y2="4.445" width="0.254" layer="1"/>
 <via x="4.572" y="4.445" extent="1-16" drill="0.35"/>
-<wire x1="4.572" y1="4.445" x2="9.144" y2="4.445" width="0.254" layer="16"/>
-<wire x1="11.303" y1="6.604" x2="11.303" y2="7.493" width="0.254" layer="16"/>
-<wire x1="9.144" y1="4.445" x2="11.303" y2="6.604" width="0.254" layer="16"/>
+<contactref element="J1" pad="4"/>
+<wire x1="10.795" y1="4.445" x2="13.843" y2="7.493" width="0.254" layer="16"/>
+<wire x1="4.572" y1="4.445" x2="10.795" y2="4.445" width="0.254" layer="16"/>
 </signal>
 <signal name="BLUE">
 <contactref element="R15" pad="2"/>
-<wire x1="16.637" y1="3.595" x2="16.217" y2="3.595" width="0.254" layer="1"/>
-<wire x1="16.217" y1="3.595" x2="15.367" y2="4.445" width="0.254" layer="1"/>
-<via x="15.367" y="4.445" extent="1-16" drill="0.35"/>
-<contactref element="J1" pad="2"/>
-<wire x1="15.367" y1="4.445" x2="10.5819875" y2="4.445" width="0.254" layer="16"/>
-<wire x1="10.5819875" y1="4.445" x2="10.05349375" y2="3.91650625" width="0.254" layer="16"/>
-<via x="10.05349375" y="3.91650625" extent="1-16" drill="0.35"/>
-<wire x1="10.05349375" y1="3.91650625" x2="8.763" y2="5.207" width="0.254" layer="1"/>
-<wire x1="8.763" y1="5.207" x2="8.763" y2="7.493" width="0.254" layer="1"/>
+<wire x1="16.637" y1="3.595" x2="16.471" y2="3.595" width="0.254" layer="1"/>
+<contactref element="J1" pad="3"/>
+<wire x1="14.605" y1="5.461" x2="12.319" y2="5.461" width="0.254" layer="1"/>
+<wire x1="12.319" y1="5.461" x2="11.303" y2="6.477" width="0.254" layer="1"/>
+<wire x1="11.303" y1="6.477" x2="11.303" y2="7.493" width="0.254" layer="1"/>
+<wire x1="16.471" y1="3.595" x2="14.605" y2="5.461" width="0.254" layer="1"/>
 </signal>
 <signal name="N$5">
@@
 <mfgpreviewcolor name="substratecolor" color="0xFF786E46"/>
 </mfgpreviewcolors>
+<errors>
+</errors>
 </board>
 </drawing>
