File: eagle-files/SmartOutlet/Motherboard.sch (EAGLE design)
At the start: 36 parts, among them IC1 1117, T1 CST-1025, U1 ADS1115IDGST, U2 ESP-WROOM-32, U3 FT232RL, X1 22-23-2041, X2 22-23-2021

Commit message: Updated eagle files
Parts:
- removed X1: 22-23-2041, con-molex:22-23-2041
- added U$1: MICRO-USB, microusb:MICRO-USB
- U1: value ADS1115IDGST -> ADS1115
- renumbered LED4 to TX_LED, LED5 to RX_LED, LED6 to POWER_LED, T1 to CURRENT_TRANSFORMER
Connections:
- net +5V: now also U$1.VCC, X2-1.S; no longer X1-1.S, X2-2.S
- net BLUE: now also R16.1; no longer R17.1
- net GND: now also U$1.GND, X2-2.S; no longer X1-4.S, X2-1.S
- net GREEN: now also R17.1; no longer R16.1
- net PLUG_D+: now also U$1.D+; no longer X1-3.S
- net PLUG_D-: now also U$1.D-; no longer X1-2.S

Commit message: Updated eagle files
Connections:
- net BUTTON: now also U2.IO5; no longer U2.IO16
Changed lines of the file:
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@@
 <attribute name="VALUE" x="43.18" y="-5.08" size="1.778" layer="96" align="bottom-right"/>
 </instance>
-<instance part="SUPPLY17" gate="GND" x="58.42" y="30.48" smashed="yes">
-<attribute name="VALUE" x="56.515" y="27.305" size="1.778" layer="96"/>
+<instance part="SUPPLY17" gate="GND" x="71.12" y="30.48" smashed="yes">
+<attribute name="VALUE" x="69.215" y="27.305" size="1.778" layer="96"/>
 </instance>
 <instance part="R7" gate="G$1" x="73.66" y="-12.7" smashed="yes">
@@
 <pinref part="U2" gate="G$1" pin="GND@4"/>
 <pinref part="SUPPLY17" gate="GND" pin="GND"/>
-<wire x1="48.26" y1="33.02" x2="58.42" y2="33.02" width="0.1524" layer="91"/>
+<wire x1="48.26" y1="33.02" x2="71.12" y2="33.02" width="0.1524" layer="91"/>
 </segment>
 <segment>
@@
 </segment>
 <segment>
-<pinref part="U2" gate="G$1" pin="IO16"/>
-<wire x1="48.26" y1="20.32" x2="50.8" y2="20.32" width="0.1524" layer="91"/>
-<label x="50.8" y="20.32" size="1.778" layer="95" xref="yes"/>
-</segment>
-</net>
+<pinref part="U2" gate="G$1" pin="IO5"/>
+<wire x1="48.26" y1="25.4" x2="50.8" y2="25.4" width="0.1524" layer="91"/>
+<label x="50.8" y="25.4" size="1.778" layer="95" xref="yes"/>
+</segment>
+</net>

Commit message: Added daughter board and edited motherboard
Parts:
- removed LED1, LED2: (no value), adafruit:LEDCHIP-LED0603
- removed R6: 10k, rcl:R-EU_R0603
- removed S2: MOMENTARY-SWITCH-SPST-PTH-6.0MM, SparkFun-Switches:MOMENTARY-SWITCH-SPST-PTH-6.0MM
- removed U$1: MICRO-USB, microusb:MICRO-USB
- added D1: (no value), adafruit:DIODE_SOD-123FL
- added K1: SRD-05VDC-SL-C, SRD-05VDC-SL-C:SRD-05VDC-SL-C
- added K2: 68610414122, 4_pin_smd_connector:68610414122
- added LED3: (no value), adafruit_custom:LEDCHIP-LED0603
- added OK1: PC817, optocoupler:PC817
- added Q1: (no value), semicon-smd-ipc:NPN-TRANSISTOR_SOT23
- added R5: 1k, rcl:R-EU_R0603
- added U$2: ZX62D-B-5P8, j_usb_hirose_zx62d-b-5p8:ZX62D-B-5P8
- added X1: (no value), con-wago-500:W237-102
- C20, C21: value 100nF -> 0.1uF; device SparkFun-Capacitors:0.1UF-0603-100V-10% -> SparkFun-Capacitors:0.1UF-0603-25V-(+80/-20%)
- POWER_LED, RX_LED, TX_LED: device adafruit:LEDCHIP-LED0603 -> adafruit_custom:LEDCHIP-LED0603
- R1, R2, R3, R4: device microbuilder:RESISTOR0805 -> rcl:R-EU_R0603
- R10, R11, R7, R8, R9: device eagle-ltspice:RR0603 -> rcl:R-EU_R0603
- R16: value 1k -> 510; device adafruit:R-US_R0603 -> rcl:R-EU_R0603
- R17: device adafruit:R-US_R0603 -> rcl:R-EU_R0603
Connections:
- removed net N$5: LED1.A, R17.2
- removed net N$6: LED2.A, R16.2
- new net N$1: LED3.A, OK1.C
- new net N$2: OK1.A, R17.1
- new net N$4: OK1.EMIT, R16.1
- new net N$7: Q1.B, R16.2
- new net N$8: D1.A, K1.A2, Q1.C
- new net POWER_IN: K1.COM, X1-2.KL
- new net POWER_SWITCHED: K1.NC, X1-1.KL
- new net RELAY: LED3.C, U2.IO17
- net +5V: now also D1.C, K1.A1, OK1.COL, U$2.1, X2-2.S; no longer U$1.VCC, X2-1.S
- net 3.3V: now also R17.2, R5.1; no longer R6.2
- net BLUE: now also K2.3; no longer R16.1
- net BUTTON: now also K2.1, R5.2, U2.IO27; no longer R6.1, S2.2, U2.IO5
- net GND: now also K2.4, Q1.E, U$2.5, X2-1.S; no longer LED1.C, LED2.C, S2.1, U$1.GND, X2-2.S
- net GREEN: now also K2.2; no longer R17.1
- net PLUG_D+: now also U$2.3; no longer U$1.D+
- net PLUG_D-: now also U$2.2; no longer U$1.D-
Other:
- moved on the sheet: C1, C18, C19, C2, C20, C21, CURRENT_TRANSFORMER, FB1, FB2, I1, R1, R2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

Commit message: Updated PCB design
Parts:
- removed CURRENT_TRANSFORMER: CST-1025, CST-1025:CST-1025
- removed I1: 0A, ngspice-simulation:CURRENT
- removed S3: MOMENTARY-SWITCH-SPST-SMD-6.0X3.5MM, SparkFun-Switches:MOMENTARY-SWITCH-SPST-SMD-6.0X3.5MM
- added C3: 0.1uF, SparkFun-Capacitors:0.1UF-0603-25V-(+80/-20%)
- added C4: 1nF, SparkFun-Capacitors:1.0NF/1000PF-0603-50V-10%
- added S2: TL1015AF160QG, small_tactile_switch:TL1015AF160QG
- added U4: ACS712ELCTR-20A-T, ACS712ELCTR-20A-T:ACS712ELCTR-20A-T
- S1: value MOMENTARY-SWITCH-SPST-SMD-6.0X3.5MM -> TL1015AF160QG; device SparkFun-Switches:MOMENTARY-SWITCH-SPST-SMD-6.0X3.5MM -> small_tactile_switch:TL1015AF160QG
- renumbered LED3 to RELAY
Connections:
- net N$8 renamed RELAY_GND
- removed net DIFF_INPUT_1: CURRENT_TRANSFORMER.1, U1.AIN0
- removed net DIFF_INPUT_2: CURRENT_TRANSFORMER.2, U1.AIN1
- removed net N$14: I1.-
- removed net N$15: I1.+
- new net ACS_FILTER: C4.1, U4.FILTER
- new net CURRENT_SENSOR: U1.AIN0, U4.VIOUT
- new net POWER_OUT: U4.IP-, X1-2.KL
- net +5V: now also C2.P$1, C3.1, FB1.P$1, U4.VCC, X2-1.S; no longer X2-2.S
- net 3.3V: no longer C2.P$1, FB1.P$1
- net BLUE: now also K2.2, U2.IO33; no longer K2.3, U2.IO32
- net BUTTON: now also K2.3, U2.IO26; no longer K2.1, U2.IO27
- net DTR: now also S1.1; no longer S3.1
- net GND: now also C3.2, C4.2, S2.2, U4.GND, X2-2.S; no longer S3.2, X2-1.S
- net GREEN: now also K2.1, U2.IO32; no longer K2.2, U2.IO33
- net POWER_IN: now also K1.NC, X1-1.KL; no longer K1.COM, X1-2.KL
- net POWER_SWITCHED: now also K1.COM, U4.IP+; no longer K1.NC, X1-1.KL
- net RTS: now also S2.1; no longer S1.1
Other:
- note added: "Connectors for AC-DC converter"
- note removed: "Connectors for AC-DC"
- note removed: "The current source represents the current being drawn from the outlet"
- moved on the sheet: D1, R5
